File: dimmer-pcb/dimmer-pcb.kicad_sch (KiCad schematic)
At the start: 13 parts, among them Q1 BT136, U1 PC817, U3 MOC3021M

Commit message: Add files via upload
Parts:
- J3: value (none) -> Conn_01x04; footprint Connector_PinHeader_1.00mm:PinHeader_1x04_P1.00mm_Vertical -> Connector_PinHeader_2.54mm:PinHeader_1x04_P2.54mm_Vertical
Changed lines of the file:
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@@
 		)
 		(instances
-			(project "dimmer"
+			(project "dimmer-pcb"
 				(path "/5daeae09-3001-4f2f-87f2-5cc963082acc"
 					(reference "R2")
@@
 		)
 		(instances
-			(project "dimmer"
+			(project "dimmer-pcb"
 				(path "/5daeae09-3001-4f2f-87f2-5cc963082acc"
 					(reference "J1")
@@
 		)
 		(instances
-			(project "dimmer"
+			(project "dimmer-pcb"
 				(path "/5daeae09-3001-4f2f-87f2-5cc963082acc"
 					(reference "#PWR04")
@@
 		)
 		(instances
-			(project "dimmer"
+			(project "dimmer-pcb"
 				(path "/5daeae09-3001-4f2f-87f2-5cc963082acc"
 					(reference "BR1")
@@
 		)
 		(instances
-			(project "dimmer"
+			(project "dimmer-pcb"
 				(path "/5daeae09-3001-4f2f-87f2-5cc963082acc"
 					(reference "U3")
@@
 		)
 		(instances
-			(project "dimmer"
+			(project "dimmer-pcb"
 				(path "/5daeae09-3001-4f2f-87f2-5cc963082acc"
 					(reference "R3")
-					(unit 1)
-				)
-			)
-		)
-	)
-	(symbol
-		(lib_id "Connector_Generic:Conn_01x04")
-		(at 127 120.65 0)
-		(unit 1)
-		(body_style 1)
-		(exclude_from_sim no)
-		(in_bom yes)
-		(on_board yes)
-		(in_pos_files yes)
-		(dnp no)
-		(fields_autoplaced yes)
-		(property "Reference" "J3"
-			(at 129.54 121.9199 0)
-			(show_name no)
-			(do_not_autoplace no)
-			(effects
-				(font
-					(size 1.27 1.27)
-				)
-				(justify left)
-			)
-		)
-		(property "Value" ""
-			(at 129.54 123.1899 0)
-			(show_name no)
-			(do_not_autoplace no)
-			(effects
-				(font
-					(size 1.27 1.27)
-				)
-				(justify left)
-			)
-		)
-		(property "Footprint" "Connector_PinHeader_1.00mm:PinHeader_1x04_P1.00mm_Vertical"
-			(at 127 120.65 0)
-			(hide yes)
-			(show_name no)
-			(do_not_autoplace no)
-			(effects
-				(font
-					(size 1.27 1.27)
-				)
-			)
-		)
-		(property "Datasheet" ""
-			(at 127 120.65 0)
-			(hide yes)
-			(show_name no)
-			(do_not_autoplace no)
-			(effects
-				(font
-					(size 1.27 1.27)
-				)
-			)
-		)
-		(property "Description" "Generic connector, single row, 01x04, script generated (kicad-library-utils/schlib/autogen/connector/)"
-			(at 127 120.65 0)
-			(hide yes)
-			(show_name no)
-			(do_not_autoplace no)
-			(effects
-				(font
-					(size 1.27 1.27)
-				)
-			)
-		)
-		(pin "3"
-		)
-		(pin "2"
-		)
-		(pin "1"
-		)
-		(pin "4"
-		)
-		(instances
-			(project "dimmer"
-				(path "/5daeae09-3001-4f2f-87f2-5cc963082acc"
-					(reference "J3")
 					(unit 1)
 				)
@@
 		)
 		(instances
-			(project "dimmer"
+			(project "dimmer-pcb"
 				(path "/5daeae09-3001-4f2f-87f2-5cc963082acc"
 					(reference "U1")
@@
 		)
 		(instances
-			(project "dimmer"
+			(project "dimmer-pcb"
 				(path "/5daeae09-3001-4f2f-87f2-5cc963082acc"
 					(reference "#PWR02")
@@
 		)
 		(instances
-			(project "dimmer"
+			(project "dimmer-pcb"
 				(path "/5daeae09-3001-4f2f-87f2-5cc963082acc"
 					(reference "R4")
+					(unit 1)
+				)
+			)
+		)
+	)
+	(symbol
+		(lib_id "Connector_Generic:Conn_01x04")
+		(at 127 120.65 0)
+		(unit 1)
+		(body_style 1)
+		(exclude_from_sim no)
+		(in_bom yes)
+		(on_board yes)
+		(in_pos_files yes)
+		(dnp no)
+		(fields_autoplaced yes)
+		(property "Reference" "J3"
+			(at 129.54 120.6499 0)
+			(show_name no)
+			(do_not_autoplace no)
+			(effects
+				(font
+					(size 1.27 1.27)
+				)
+				(justify left)
+			)
+		)
+		(property "Value" "Conn_01x04"
+			(at 129.54 123.1899 0)
+			(show_name no)
+			(do_not_autoplace no)
+			(effects
+				(font
+					(size 1.27 1.27)
+				)
+				(justify left)
+			)
+		)
+		(property "Footprint" "Connector_PinHeader_2.54mm:PinHeader_1x04_P2.54mm_Vertical"
+			(at 127 120.65 0)
+			(hide yes)
+			(show_name no)
+			(do_not_autoplace no)
+			(effects
+				(font
+					(size 1.27 1.27)
+				)
+			)
+		)
+		(property "Datasheet" ""
+			(at 127 120.65 0)
+			(hide yes)
+			(show_name no)
+			(do_not_autoplace no)
+			(effects
+				(font
+					(size 1.27 1.27)
+				)
+			)
+		)
+		(property "Description" "Generic connector, single row, 01x04, script generated (kicad-library-utils/schlib/autogen/connector/)"
+			(at 127 120.65 0)
+			(hide yes)
+			(show_name no)
+			(do_not_autoplace no)
+			(effects
+				(font
+					(size 1.27 1.27)
+				)
+			)
+		)
+		(pin "1"
+		)
+		(pin "2"
+		)
+		(pin "3"
+		)
+		(pin "4"
+		)
+		(instances
+			(project "dimmer-pcb"
+				(path "/5daeae09-3001-4f2f-87f2-5cc963082acc"
+					(reference "J3")
 					(unit 1)
 				)
@@
 		)
 		(instances
-			(project "dimmer"
+			(project "dimmer-pcb"
 				(path "/5daeae09-3001-4f2f-87f2-5cc963082acc"
 					(reference "#PWR05")
@@
 		)
 		(instances
-			(project "dimmer"
+			(project "dimmer-pcb"
 				(path "/5daeae09-3001-4f2f-87f2-5cc963082acc"
 					(reference "R1")
@@
 		)
 		(instances
-			(project "dimmer"
+			(project "dimmer-pcb"
 				(path "/5daeae09-3001-4f2f-87f2-5cc963082acc"
 					(reference "#PWR01")
@@
 		)
 		(instances
-			(project "dimmer"
+			(project "dimmer-pcb"
 				(path "/5daeae09-3001-4f2f-87f2-5cc963082acc"
 					(reference "J2")
@@
 		)
 		(instances
-			(project "dimmer"
+			(project "dimmer-pcb"
 				(path "/5daeae09-3001-4f2f-87f2-5cc963082acc"
 					(reference "C1")
@@
 		)
 		(instances
-			(project "dimmer"
+			(project "dimmer-pcb"
 				(path "/5daeae09-3001-4f2f-87f2-5cc963082acc"
 					(reference "R5")
@@
 		)
 		(instances
-			(project "dimmer"
+			(project "dimmer-pcb"
 				(path "/5daeae09-3001-4f2f-87f2-5cc963082acc"
 					(reference "Q1")
@@
 		)
 		(instances
-			(project "dimmer"
+			(project "dimmer-pcb"
 				(path "/5daeae09-3001-4f2f-87f2-5cc963082acc"
 					(reference "#PWR03")
