File: dimmer-pcb/dimmer-pcb.kicad_pcb (KiCad board)
At the start: 2 copper layers, 13 parts, among them Q1 BT136, U1 PC817, U3 MOC3021M

Commit message: Add files via upload
Parts:
- J3: value ~ -> Conn_01x04; footprint Connector_PinHeader_1.00mm:PinHeader_1x04_P1.00mm_Vertical -> Connector_PinHeader_2.54mm:PinHeader_1x04_P2.54mm_Vertical
- moved J3 7.34 mm to (138.5, 111.2)
- moved R4 4.81 mm to (132.5, 113.0)
Routing:
- net Net-(J3-Pin_3): track 25.3 -> 17.9 mm, vias 2 -> 0
- net +5V: track 3.50 -> 7.29 mm
- net GND: track 32.7 -> 34.9 mm
- net Net-(J3-Pin_4): track 7.91 -> 9.41 mm

Commit message: Add files via upload
Other:
- board text added: "SASoftwareS"
Changed lines of the file:
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@@
 		(filling no)
 		(pcbplotparams
-			(layerselection 0x00000000_00000000_55555555_5755f5ff)
+			(layerselection 0x00000000_00000000_55555555_55555574)
 			(plot_on_all_layers_selection 0x00000000_00000000_00000000_00000000)
 			(disableapertmacros no)
@@
 			(crossoutdnponfab yes)
 			(subtractmaskfromsilk no)
-			(outputformat 1)
+			(outputformat 4)
 			(mirror no)
-			(drillshape 0)
+			(drillshape 2)
 			(scaleselection 1)
 			(outputdirectory "")
@@
 		(layer "B.Cu")
 	)
+	(gr_text "SASoftwareS"
+		(at 135.5 122 0)
+		(layer "B.Cu")
+		(effects
+			(font
+				(size 1 1)
+				(thickness 0.2)
+				(bold yes)
+			)
+			(justify left bottom mirror)
+		)
+	)
+	(gr_text "SASoftwareS"
+		(at 126 122 0)
+		(layer "F.SilkS")
+		(effects
+			(font
+				(size 1 1)
+				(thickness 0.1)
+			)
+			(justify left bottom)
+		)
+	)
+	(segment
+		(start 102.5 120.75)
+		(end 102.5 121)
+		(width 2)
+		(layer "F.Cu")
+		(net "Net-(J1-Pin_1)")
+	)
+	(segment
+		(start 102.5 114)
+		(end 102.5 120.75)
+		(width 2)
+		(layer "F.Cu")
+		(net "Net-(J1-Pin_1)")
+	)
+	(via
+		(at 102.5 121)
+		(size 1)
+		(drill 0.3)
+		(layers "F.Cu" "B.Cu")
+		(net "Net-(J1-Pin_1)")
+	)
+	(via
+		(at 102.5 114)
+		(size 1)
+		(drill 0.3)
+		(layers "F.Cu" "B.Cu")
+		(net "Net-(J1-Pin_1)")
+	)
+	(segment
+		(start 102.5 122.41)
+		(end 104.05 123.96)
+		(width 2)
+		(layer "B.Cu")
+		(net "Net-(J1-Pin_1)")
+	)
+	(segment
+		(start 111.29 123.96)
+		(end 111.75 123.5)
+		(width 2)
+		(layer "B.Cu")
+		(net "Net-(J1-Pin_1)")
+	)
+	(segment
+		(start 102.5 112.5)
+		(end 102.5 114)
+		(width 2)
+		(layer "B.Cu")
+		(net "Net-(J1-Pin_1)")
+	)
+	(segment
+		(start 104.05 123.96)
+		(end 111.29 123.96)
+		(width 2)
+		(layer "B.Cu")
+		(net "Net-(J1-Pin_1)")
+	)
+	(segment
+		(start 95.5 112.5)
+		(end 102.5 112.5)
+		(width 2.5)
+		(layer "B.Cu")
+		(net "Net-(J1-Pin_1)")
+	)
+	(segment
+		(start 102.5 121)
+		(end 102.5 122.41)
+		(width 2)
+		(layer "B.Cu")
+		(net "Net-(J1-Pin_1)")
+	)
+	(segment
+		(start 110.825 117.5)
+		(end 110.875 117.55)
+		(width 2.5)
+		(layer "B.Cu")
+		(net "Net-(J1-Pin_2)")
+	)
+	(segment
+		(start 95.5 117.5)
+		(end 110.825 117.5)
+		(width 2.5)
+		(layer "B.Cu")
+		(net "Net-(J1-Pin_2)")
+	)
+	(segment
+		(start 95.5 117.5)
+		(end 95.5 124)
+		(width 2.5)
+		(layer "B.Cu")
+		(net "Net-(J1-Pin_2)")
+	)
 	(segment
 		(start 133.31 111.19)
@@
 	)
 	(segment
-		(start 102.5 120.75)
-		(end 102.5 121)
-		(width 2)
-		(layer "F.Cu")
-		(net "Net-(J1-Pin_1)")
-	)
-	(segment
-		(start 102.5 114)
-		(end 102.5 120.75)
-		(width 2)
-		(layer "F.Cu")
-		(net "Net-(J1-Pin_1)")
-	)
-	(via
-		(at 102.5 121)
-		(size 1)
-		(drill 0.3)
-		(layers "F.Cu" "B.Cu")
-		(net "Net-(J1-Pin_1)")
-	)
-	(via
-		(at 102.5 114)
-		(size 1)
-		(drill 0.3)
-		(layers "F.Cu" "B.Cu")
-		(net "Net-(J1-Pin_1)")
-	)
-	(segment
-		(start 102.5 122.41)
-		(end 104.05 123.96)
-		(width 2)
-		(layer "B.Cu")
-		(net "Net-(J1-Pin_1)")
-	)
-	(segment
-		(start 111.29 123.96)
-		(end 111.75 123.5)
-		(width 2)
-		(layer "B.Cu")
-		(net "Net-(J1-Pin_1)")
-	)
-	(segment
-		(start 102.5 112.5)
-		(end 102.5 114)
-		(width 2)
-		(layer "B.Cu")
-		(net "Net-(J1-Pin_1)")
-	)
-	(segment
-		(start 104.05 123.96)
-		(end 111.29 123.96)
-		(width 2)
-		(layer "B.Cu")
-		(net "Net-(J1-Pin_1)")
-	)
-	(segment
-		(start 95.5 112.5)
-		(end 102.5 112.5)
-		(width 2.5)
-		(layer "B.Cu")
-		(net "Net-(J1-Pin_1)")
-	)
-	(segment
-		(start 102.5 121)
-		(end 102.5 122.41)
-		(width 2)
-		(layer "B.Cu")
-		(net "Net-(J1-Pin_1)")
-	)
-	(segment
-		(start 110.825 117.5)
-		(end 110.875 117.55)
-		(width 2.5)
-		(layer "B.Cu")
-		(net "Net-(J1-Pin_2)")
-	)
-	(segment
-		(start 95.5 117.5)
-		(end 110.825 117.5)
-		(width 2.5)
-		(layer "B.Cu")
-		(net "Net-(J1-Pin_2)")
-	)
-	(segment
-		(start 95.5 117.5)
-		(end 95.5 124)
-		(width 2.5)
-		(layer "B.Cu")
-		(net "Net-(J1-Pin_2)")
-	)
-	(segment
 		(start 112.4 131.2)
 		(end 112.4 131.15)
@@
 		(start 138.415 130.54)
 		(end 138.455 130.5)
-		(width 1.5)
+		(width 0.5)
 		(layer "B.Cu")
 		(net "Net-(R5-Pad1)")
@@
 		(start 134.81 130.54)
 		(end 138.415 130.54)
-		(width 1.5)
+		(width 0.5)
 		(layer "B.Cu")
 		(net "Net-(R5-Pad1)")

Commit message: Add files via upload
Parts:
- U3: value MOC3021M -> MOC3021
- renumbered BR1 to DB107
Routing:
- net Net-(J1-Pin_1): track 27.0 -> 42.8 mm, vias 2 -> 0
Changed lines of the file:
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@@
 			(at 2.25 -5.12 90)
 			(layer "F.SilkS")
+			(hide yes)
 			(effects
 				(font
@@
 			(at 0 -2.38 0)
 			(layer "F.SilkS")
+			(hide yes)
 			(effects
 				(font
@@
 			(at 2.54 -4.1 90)
 			(layer "F.SilkS")
+			(hide yes)
 			(effects
 				(font
@@
 			(at 2.54 -2.37 0)
 			(layer "F.SilkS")
+			(hide yes)
 			(effects
 				(font
@@
 			(at 1.27 -2.37 90)
 			(layer "F.SilkS")
+			(hide yes)
 			(effects
 				(font
@@
 			(at 1.27 -2.37 0)
 			(layer "F.SilkS")
+			(hide yes)
 			(effects
 				(font
@@
 			(at 3.81 -2.33 0)
 			(layer "F.SilkS")
+			(hide yes)
 			(effects
 				(font
@@
 			)
 		)
-		(property "Value" "MOC3021M"
+		(property "Value" "MOC3021"
 			(at 3.81 7.41 0)
 			(layer "F.Fab")
@@
 			(at 3.81 -2.33 90)
 			(layer "F.SilkS")
+			(hide yes)
 			(effects
 				(font
@@
 			(at 5 -3.75 0)
 			(layer "F.SilkS")
+			(hide yes)
 			(effects
 				(font
@@
 		)
 		(property "Value" "104J"
-			(at 5 3.75 0)
+			(at 4.75 1.5 0)
 			(layer "F.Fab")
 			(effects
@@
 			(at 2.25 -5.12 90)
 			(layer "F.SilkS")
+			(hide yes)
 			(effects
 				(font
@@
 		(layer "F.Cu")
 		(at 115 115 180)
-		(property "Reference" "BR1"
+		(property "Reference" "DB107"
 			(at -0.645 -5.635 0)
 			(layer "F.SilkS")
+			(hide yes)
 			(effects
 				(font
@@
 		)
 		(property "Value" "DB107"
-			(at 10.785 5.635 0)
+			(at -0.25 -2 0)
 			(layer "F.Fab")
 			(effects
@@
 			(at 1.27 -2.37 90)
 			(layer "F.SilkS")
+			(hide yes)
 			(effects
 				(font
@@
 			(at 2.54 -2.37 0)
 			(layer "F.SilkS")
+			(hide yes)
 			(effects
 				(font
@@
 	)
 	(segment
-		(start 102.5 120.75)
-		(end 102.5 121)
+		(start 114.5 120.75)
+		(end 111.75 123.5)
 		(width 2)
-		(layer "F.Cu")
+		(layer "B.Cu")
 		(net "Net-(J1-Pin_1)")
 	)
 	(segment
-		(start 102.5 114)
-		(end 102.5 120.75)
+		(start 102.5 112)
+		(end 105 109.5)
 		(width 2)
-		(layer "F.Cu")
-		(net "Net-(J1-Pin_1)")
-	)
-	(via
-		(at 102.5 121)
-		(size 1)
-		(drill 0.3)
-		(layers "F.Cu" "B.Cu")
+		(layer "B.Cu")
 		(net "Net-(J1-Pin_1)")
 	)
-	(via
-		(at 102.5 114)
-		(size 1)
-		(drill 0.3)
-		(layers "F.Cu" "B.Cu")
+	(segment
+		(start 111.29 123.96)
+		(end 111.75 123.5)
+		(width 2)
+		(layer "B.Cu")
 		(net "Net-(J1-Pin_1)")
 	)
 	(segment
-		(start 102.5 122.41)
-		(end 104.05 123.96)
+		(start 113.25 109.5)
+		(end 114.5 110.75)
 		(width 2)
 		(layer "B.Cu")
@@
 	)
 	(segment
-		(start 111.29 123.96)
-		(end 111.75 123.5)
+		(start 104.05 123.96)
+		(end 111.29 123.96)
 		(width 2)
 		(layer "B.Cu")
@@
 	)
 	(segment
-		(start 102.5 112.5)
-		(end 102.5 114)
+		(start 114.5 110.75)
+		(end 114.5 120.75)
 		(width 2)
 		(layer "B.Cu")
@@
 	)
 	(segment
-		(start 104.05 123.96)
-		(end 111.29 123.96)
+		(start 102.5 112.5)
+		(end 102.5 112)
 		(width 2)
 		(layer "B.Cu")
@@
 	)
 	(segment
-		(start 102.5 121)
-		(end 102.5 122.41)
+		(start 105 109.5)
+		(end 113.25 109.5)
 		(width 2)
 		(layer "B.Cu")

Commit message: Add files via upload
Parts:
- moved J3 7.39 mm to (138.5, 118.6), turned to 180 degrees
- moved R4 5.59 mm to (132.5, 118.5), turned to 90 degrees
Routing:
- net Net-(J3-Pin_3): track 17.9 -> 30.8 mm
- net Net-(J3-Pin_4): track 9.41 -> 19.1 mm
- net GND: track 34.9 -> 31.3 mm
- net +5V: track 7.29 -> 6.01 mm
